Commit message: Update myrobot.xacro

File: urdf/myrobot.xacro (robot description, xacro)
@@ -23,7 +23,7 @@
    <link name="base_footprint" />
    <joint name="base_footprint_joint" type="fixed">
-      <parent link="base_link" />
-      <child link="base_footprint" />
-      <origin xyz="0 0 -0.185" rpy="0 0 0" />
+      <child link="base_link" />
+      <parent link="base_footprint" />
+      <origin xyz="0 0 0.185" rpy="0 0 0" />
    </joint>
    <link name="front_caster">

Commit message: Update myrobot.xacro

File: urdf/myrobot.xacro (robot description, xacro)
@@ -1,5 +1,5 @@
 <?xml version="1.0" encoding="UTF-8"?>
 <robot xmlns:xacro="http://ros.org/wiki/xacro" name="tortoisebot">
-   <xacro:include filename="$(find lidar-2d-mapping)/urdf/myrobot.gazebo" />
+   <xacro:include filename="$(find lidar_2d_mapping)/urdf/myrobot.gazebo" />
    <link name="base_link">
       <visual>
@@ -146,5 +146,5 @@
          <origin xyz="0 0 0" rpy="0 0 0" />
          <geometry>
-            <mesh filename="file://$(find lidar-2d-mapping)/meshes/lidar.dae" />
+            <mesh filename="file://$(find lidar_2d_mapping)/meshes/lidar.dae" />
          </geometry>
       </visual>
